Commit message: 2026-09-30 own robot: rigid chassis, guessed masses (3 kg total, 0.1 kg rotating wheel), motor guess
generate_mecanum_robot.py: RobotParams.front_axle (False = rigid chassis, all wheels on base_link); the default
(FUJI) robot.urdf is byte-identical. Own robot: 41 links, 3.0 kg (chassis incl. motors 2.6 kg, hub 55 g,
rollers 9 x 5 g), rubber-coated rollers. Motor guess (12 V ~1:30 gear motor: 35 rad/s no-load, 1.5 Nm stall,
0.6 Nm continuous, 9e-4 kg m^2 reflected inertia) recorded in robot_config.json for the robot cfg.

Co-Authored-By: Claude Opus 5.5 <noreply@anthropic.com>

File: assets/robots/own_mecanum/robot.urdf (robot description, URDF)
Before this commit: robot mecanum_rollers, 42 links, 41 joints
Links:
- removed link front_axle
- link base_link: mass 1.5335 -> 2.6
- link front_left_roller_00: mass 0.00375 -> 0.005
- link front_left_roller_01: mass 0.00375 -> 0.005
- link front_left_roller_02: mass 0.00375 -> 0.005
- link front_left_roller_03: mass 0.00375 -> 0.005
- link front_left_roller_04: mass 0.00375 -> 0.005
- link front_left_roller_05: mass 0.00375 -> 0.005
- link front_left_roller_06: mass 0.00375 -> 0.005
- link front_left_roller_07: mass 0.00375 -> 0.005
- link front_left_roller_08: mass 0.00375 -> 0.005
- link front_left_wheel: mass 0.04378 -> 0.055
- link front_right_roller_00: mass 0.00375 -> 0.005
- link front_right_roller_01: mass 0.00375 -> 0.005
- link front_right_roller_02: mass 0.00375 -> 0.005
- link front_right_roller_03: mass 0.00375 -> 0.005
- link front_right_roller_04: mass 0.00375 -> 0.005
- link front_right_roller_05: mass 0.00375 -> 0.005
- link front_right_roller_06: mass 0.00375 -> 0.005
- link front_right_roller_07: mass 0.00375 -> 0.005
- link front_right_roller_08: mass 0.00375 -> 0.005
- link front_right_wheel: mass 0.04378 -> 0.055
- link rear_left_roller_00: mass 0.00375 -> 0.005
- link rear_left_roller_01: mass 0.00375 -> 0.005
- link rear_left_roller_02: mass 0.00375 -> 0.005
- link rear_left_roller_03: mass 0.00375 -> 0.005
- link rear_left_roller_04: mass 0.00375 -> 0.005
- link rear_left_roller_05: mass 0.00375 -> 0.005
- link rear_left_roller_06: mass 0.00375 -> 0.005
- link rear_left_roller_07: mass 0.00375 -> 0.005
- link rear_left_roller_08: mass 0.00375 -> 0.005
- link rear_left_wheel: mass 0.04378 -> 0.055
- link rear_right_roller_00: mass 0.00375 -> 0.005
- link rear_right_roller_01: mass 0.00375 -> 0.005
- link rear_right_roller_02: mass 0.00375 -> 0.005
- link rear_right_roller_03: mass 0.00375 -> 0.005
- link rear_right_roller_04: mass 0.00375 -> 0.005
- link rear_right_roller_05: mass 0.00375 -> 0.005
- link rear_right_roller_06: mass 0.00375 -> 0.005
- link rear_right_roller_07: mass 0.00375 -> 0.005
- link rear_right_roller_08: mass 0.00375 -> 0.005
- link rear_right_wheel: mass 0.04378 -> 0.055
Joints:
- removed joint front_axle_joint
- joint front_left_wheel_joint: origin xyz=0 0.1526 0 -> xyz=0.064 0.1526 -0.0415; parent front_axle -> base_link
- joint front_right_wheel_joint: origin xyz=0 -0.1526 0 -> xyz=0.064 -0.1526 -0.0415; parent front_axle -> base_link

Commit message: 2026-09-30 own robot: CAD chassis (Fusion base_link.stl) instead of the box
generate_mecanum_robot.py: optional chassis mesh (RobotParams.chassis_mesh_*): vertex-clustering decimated visual
(2 mm cell: 951627 -> 233023 triangles, visually identical at video resolution), convex hull as collider
(656 triangles), mesh origin / orientation and full inertia tensor with COM. FUJI robot.urdf byte-identical.
Own robot: chassis rotated 180 deg about z (CAD front = -x), origin 64.8 mm below the box center (wheels at the
assembly positions), Fusion COM (+16 mm in x) and inertia scaled to 2.6 kg.
Drive test: forward -1.2 %, sideways -4.5 %, diagonal -0.9 % (wz drift -0.013 rad/s), rotation -2.4 % (vy 0.015 m/s).

Co-Authored-By: Claude Opus 5.5 <noreply@anthropic.com>

File: assets/robots/own_mecanum/robot.urdf (robot description, URDF)
Before this commit: robot mecanum_rollers, 41 links, 40 joints
Links:
- link base_link: geometry collision mesh filename=meshes/chassis_collision.stl; visual mesh filename=meshes/chassis_visual.stl
